Commit message: changed example 11 to work with ackermann controller

File: example_11/description/ros2_control/carlikebot.ros2_control.xacro (robot description, xacro)
@@ -8,5 +8,5 @@
         <param name="example_param_hw_stop_duration_sec">3.0</param>
       </hardware>
-      <joint name="${prefix}virtual_front_wheel_joint">
+      <!-- <joint name="${prefix}virtual_front_wheel_joint">
         <command_interface name="position"/>
         <state_interface name="position"/>
@@ -16,4 +16,24 @@
         <state_interface name="velocity"/>
         <state_interface name="position"/>
+      </joint> -->
+      <!-- Front steering joints (position control) -->
+      <joint name="${prefix}front_left_wheel_joint">
+        <command_interface name="position"/>
+        <state_interface name="position"/>
+      </joint>
+      <joint name="${prefix}front_right_wheel_joint">
+        <command_interface name="position"/>
+        <state_interface name="position"/>
+      </joint>
+      <!-- Rear wheel joints (velocity + position feedback) -->
+      <joint name="${prefix}rear_left_wheel_joint">
+        <command_interface name="velocity"/>
+        <state_interface name="velocity"/>
+        <state_interface name="position"/>
+      </joint>
+      <joint name="${prefix}rear_right_wheel_joint">
+        <command_interface name="velocity"/>
+        <state_interface name="velocity"/>
+        <state_interface name="position"/>
       </joint>
     </ros2_control>

File: ros2_control_demo_description/carlikebot/urdf/carlikebot_description.urdf.xacro (robot description, xacro)
@@ -48,5 +48,5 @@
     <!-- rear wheels -->
     <!-- virtual rear wheel -->
-    <link name="${prefix}virtual_rear_wheel">
+    <!-- <link name="${prefix}virtual_rear_wheel">
       <visual>
         <origin xyz="0 0 0" rpy="${PI/2} 0 ${PI/2}"/>
@@ -64,5 +64,5 @@
       <limit effort="100.0" velocity="100.0"/>
       <dynamics damping="0.2"/>
-    </joint>
+    </joint> -->
     <!-- rear right wheel -->
     <link name="${prefix}rear_right_wheel">
@@ -96,5 +96,5 @@
       <limit effort="100.0" velocity="100.0"/>
       <dynamics damping="0.2"/>
-      <mimic joint="${prefix}virtual_rear_wheel_joint" multiplier="1.0" offset="0.0"/>
+      <!-- <mimic joint="${prefix}virtual_rear_wheel_joint" multiplier="1.0" offset="0.0"/> -->
     </joint>
     <!-- rear left wheel -->
@@ -129,9 +129,9 @@
       <limit effort="100.0" velocity="100.0"/>
       <dynamics damping="0.2"/>
-      <mimic joint="${prefix}virtual_rear_wheel_joint" multiplier="1.0" offset="0.0"/>
+      <!-- <mimic joint="${prefix}virtual_rear_wheel_joint" multiplier="1.0" offset="0.0"/> -->
     </joint>
     <!-- front wheels -->
     <!-- virtual front wheel -->
-    <link name="${prefix}virtual_front_wheel">
+    <!-- <link name="${prefix}virtual_front_wheel">
       <visual>
         <origin xyz="0 0 0" rpy="${PI/2} 0 ${PI/2}"/>
@@ -149,5 +149,5 @@
       <limit lower="-0.4" upper="0.4" effort="100.0" velocity="10.0"/>
       <dynamics damping="0.2"/>
-    </joint>
+    </joint> -->
     <!-- front right wheel -->
     <link name="${prefix}front_right_wheel">
@@ -181,5 +181,5 @@
       <limit lower="-0.4" upper="0.4" effort="100.0" velocity="10.0"/>
       <dynamics damping="0.2"/>
-      <mimic joint="${prefix}virtual_front_wheel_joint" multiplier="1.0" offset="0.0"/>
+      <!-- <mimic joint="${prefix}virtual_front_wheel_joint" multiplier="1.0" offset="0.0"/> -->
     </joint>
     <!-- front left steering -->
@@ -214,5 +214,5 @@
       <limit lower="-0.4" upper="0.4" effort="100.0" velocity="10.0"/>
       <dynamics damping="0.2"/>
-      <mimic joint="${prefix}virtual_front_wheel_joint" multiplier="1.0" offset="0.0"/>
+      <!-- <mimic joint="${prefix}virtual_front_wheel_joint" multiplier="1.0" offset="0.0"/> -->
     </joint>
   </xacro:macro>
